File: hardware/cmdc0de-apa104.sch (EAGLE design)
At the start: 128 parts, among them IC1 ATTINY13A-SSU

Commit message: no errors board is complete?
Parts:
- APA104-1, APA104-10, APA104-11, APA104-12, APA104-13, APA104-14, APA104-15, APA104-16, APA104-17, APA104-18, APA104-19, APA104-2, APA104-20, APA104-21, APA104-22, APA104-23, APA104-24, APA104-25, APA104-26, APA104-27, APA104-28, APA104-29, APA104-3, APA104-30, APA104-31, APA104-32, APA104-33, APA104-34, APA104-35, APA104-36, APA104-37, APA104-38, APA104-39, APA104-4, APA104-40, APA104-41, APA104-42, APA104-43, APA104-44, APA104-45, APA104-46, APA104-47, APA104-48, APA104-49, APA104-5, APA104-50, APA104-51, APA104-52, APA104-53, APA104-54, APA104-55, APA104-56, APA104-57, APA104-58, APA104-59, APA104-6, APA104-60, APA104-7, APA104-8, APA104-9: device dc-26:APA104 -> name-in-lights:APA104
- C-L-10, C-L-11, C-L-12, C-L-13, C-L-14, C-L-15, C-L-16, C-L-17, C-L-18, C-L-19, C-L-2, C-L-20, C-L-21, C-L-22, C-L-23, C-L-24, C-L-25, C-L-26, C-L-27, C-L-28, C-L-29, C-L-3, C-L-30, C-L-31, C-L-32, C-L-33, C-L-34, C-L-35, C-L-36, C-L-37, C-L-38, C-L-39, C-L-4, C-L-40, C-L-41, C-L-42, C-L-43, C-L-44, C-L-45, C-L-46, C-L-47, C-L-48, C-L-49, C-L-5, C-L-50, C-L-51, C-L-52, C-L-53, C-L-54, C-L-55, C-L-56, C-L-57, C-L-58, C-L-59, C-L-6, C-L-60, C-L-7, C-L-8, C-L9: value (none) -> 15pf
- C81, C82, C83: device NameInLights:C-USC0805 -> name-in-lights:C-USC0805-VOLTERA
- J1: value (none) -> 1x8 header
- POWER-IN: value (none) -> 5V
- renumbered J2 to POWER-IN
Connections:
- removed net GPIO_APA106_DATA: J1.7
- removed net N$69: APA104-60.DOUT
- removed net VCC: C81.2, C82.2, IC1.VCC, J1.1, POWER-IN.1, R1.1
- removed net VCC5V: APA104-1.VDD, APA104-10.VDD, APA104-11.VDD, APA104-12.VDD, APA104-13.VDD, APA104-14.VDD, APA104-15.VDD, APA104-16.VDD, APA104-17.VDD, APA104-18.VDD, APA104-19.VDD, APA104-2.VDD, APA104-20.VDD, APA104-21.VDD, APA104-22.VDD, APA104-23.VDD, APA104-24.VDD, APA104-25.VDD, APA104-26.VDD, APA104-27.VDD, APA104-28.VDD, APA104-29.VDD, APA104-3.VDD, APA104-30.VDD, APA104-31.VDD, APA104-32.VDD, APA104-33.VDD, APA104-34.VDD, APA104-35.VDD, APA104-36.VDD, APA104-37.VDD, APA104-38.VDD, APA104-39.VDD, APA104-4.VDD, APA104-40.VDD, APA104-41.VDD, APA104-42.VDD, APA104-43.VDD, APA104-44.VDD, APA104-45.VDD, APA104-46.VDD, APA104-47.VDD, APA104-48.VDD, APA104-49.VDD, APA104-5.VDD, APA104-50.VDD, APA104-51.VDD, APA104-52.VDD, APA104-53.VDD, APA104-54.VDD, APA104-55.VDD, APA104-56.VDD, APA104-57.VDD, APA104-58.VDD, APA104-59.VDD, APA104-6.VDD, APA104-60.VDD, APA104-7.VDD, APA104-8.VDD, APA104-9.VDD, C-L-1.2, C-L-10.1, C-L-11.1, C-L-12.1, C-L-13.1, C-L-14.1, C-L-15.1, C-L-16.1, C-L-17.1, C-L-18.1, C-L-19.1, C-L-2.1, C-L-20.1, C-L-21.1, C-L-22.1, C-L-23.1, C-L-24.1, C-L-25.1, C-L-26.1, C-L-27.1, C-L-28.1, C-L-29.1, C-L-3.1, C-L-30.1, C-L-31.1, C-L-32.1, C-L-33.1, C-L-34.1, C-L-35.1, C-L-36.1, C-L-37.1, C-L-38.1, C-L-39.1, C-L-4.1, C-L-40.1, C-L-41.1, C-L-42.1, C-L-43.1, C-L-44.1, C-L-45.1, C-L-46.1, C-L-47.1, C-L-48.1, C-L-49.1, C-L-5.1, C-L-50.1, C-L-51.1, C-L-52.1, C-L-53.1, C-L-54.1, C-L-55.1, C-L-56.1, C-L-57.1, C-L-58.1, C-L-59.1, C-L-6.1, C-L-60.1, C-L-7.1, C-L-8.1, C-L9.1
- new net VDD: APA104-1.VDD, APA104-10.VDD, APA104-11.VDD, APA104-12.VDD, APA104-13.VDD, APA104-14.VDD, APA104-15.VDD, APA104-16.VDD, APA104-17.VDD, APA104-18.VDD, APA104-19.VDD, APA104-2.VDD, APA104-20.VDD, APA104-21.VDD, APA104-22.VDD, APA104-23.VDD, APA104-24.VDD, APA104-25.VDD, APA104-26.VDD, APA104-27.VDD, APA104-28.VDD, APA104-29.VDD, APA104-3.VDD, APA104-30.VDD, APA104-31.VDD, APA104-32.VDD, APA104-33.VDD, APA104-34.VDD, APA104-35.VDD, APA104-36.VDD, APA104-37.VDD, APA104-38.VDD, APA104-39.VDD, APA104-4.VDD, APA104-40.VDD, APA104-41.VDD, APA104-42.VDD, APA104-43.VDD, APA104-44.VDD, APA104-45.VDD, APA104-46.VDD, APA104-47.VDD, APA104-48.VDD, APA104-49.VDD, APA104-5.VDD, APA104-50.VDD, APA104-51.VDD, APA104-52.VDD, APA104-53.VDD, APA104-54.VDD, APA104-55.VDD, APA104-56.VDD, APA104-57.VDD, APA104-58.VDD, APA104-59.VDD, APA104-6.VDD, APA104-60.VDD, APA104-7.VDD, APA104-8.VDD, APA104-9.VDD, C-L-1.2, C-L-10.1, C-L-11.1, C-L-12.1, C-L-13.1, C-L-14.1, C-L-15.1, C-L-16.1, C-L-17.1, C-L-18.1, C-L-19.1, C-L-2.1, C-L-20.1, C-L-21.1, C-L-22.1, C-L-23.1, C-L-24.1, C-L-25.1, C-L-26.1, C-L-27.1, C-L-28.1, C-L-29.1, C-L-3.1, C-L-30.1, C-L-31.1, C-L-32.1, C-L-33.1, C-L-34.1, C-L-35.1, C-L-36.1, C-L-37.1, C-L-38.1, C-L-39.1, C-L-4.1, C-L-40.1, C-L-41.1, C-L-42.1, C-L-43.1, C-L-44.1, C-L-45.1, C-L-46.1, C-L-47.1, C-L-48.1, C-L-49.1, C-L-5.1, C-L-50.1, C-L-51.1, C-L-52.1, C-L-53.1, C-L-54.1, C-L-55.1, C-L-56.1, C-L-57.1, C-L-58.1, C-L-59.1, C-L-6.1, C-L-60.1, C-L-7.1, C-L-8.1, C-L9.1, C81.2, C82.2, IC1.VCC, J1.1, POWER-IN.1, R1.1
- net GPIO_APA104_DATA: now also J1.5
- net PB0-MOSI: now also J1.4; no longer J1.6
- net PB1-MISO: now also J1.3; no longer J1.5
- net PB2-SCK: now also J1.2; no longer J1.4
- net PB3: now also J1.6; no longer J1.3
- net RESET: now also J1.7; no longer J1.2
